Commit message: Initial commit: CS625 ROS2 workspace
- 24 ROS2 packages for Elite CS625 6-axis robot arm
- MoveIt 2 motion planning + ros2_control system
- Gazebo simulation support with NBV pipeline
- cs625_nbv: PoseGain-NBV next-best-view planning (new package)
- cs625_kinematics: multi-solution IK solver
- cs625_state_monitor: robot state logging and monitoring
- cs625_trajectory_tools: MoveIt planning client
- cs625_task_manager: FSM-based task supervisor
- environment_point_cloud_publisher: multi-view point cloud fusion
- workspace_pointcloud_sampler: workspace point cloud sampling
- environment_collision_generator: collision scene generation
- vision_bridge: external TCP pose bridge
- tcp_bridge: dual-layer TCP bridge (S/R + P/J/T1/T2 protocol)
- Fixed C++17 compatibility (std::numbers::pi, PIMPL destructors, nested struct defaults)
- Added sim_state_publisher for simulation mode
- Added NBV scene world (nbv_scene.sdf) and launch files

File: src/eli_cs_robot_description/urdf/cs.ros2_control.xacro (robot description, xacro)
@@ -49,7 +49,11 @@
           <param name="trajectory_port">${trajectory_port}</param>
           <param name="tf_prefix">${tf_prefix}</param>
-          <param name="servoj_gain">1000</param>
-          <param name="servoj_lookahead_time">0.03</param>
-          <param name="servoj_time">0.008</param>
+	  <param name="servoj_gain">220</param>
+	  <param name="servoj_lookahead_time">0.10</param>
+	  <param name="servoj_time">0.008</param>
+	  <param name="servoj_extrapolate_max_time">0.04</param>
+	  <param name="servoj_decelerate_time">0.04</param>
+	  <param name="servoj_hold_velocity_threshold">0.06</param>
+	  <param name="servoj_hold_stable_time">0.03</param>
           <param name="use_tool_communication">${use_tool_communication}</param>
           <param name="tool_voltage">${tool_voltage}</param>

File: src/eli_cs_robot_description/urdf/cs.urdf.xacro (robot description, xacro)
@@ -1,4 +1,4 @@
 <?xml version="1.0"?>
-<robot xmlns:xacro="http://wiki.ros.org/xacro" name="$(arg name)">
+<robot xmlns:xacro="http://wiki.ros.org/xacro" name="cs625">
    <!-- robot name parameter -->
    <xacro:arg name="name" default="cs625"/>
@@ -7,5 +7,5 @@
    <!-- possible 'cs_type' values: cs63, cs66, cs612, cs616, cs620, cs625 -->
    <!-- the default value should raise an error in case this was called without defining the type -->
-   <xacro:arg name="cs_type" default="cs63"/>
+   <xacro:arg name="cs_type" default="cs625"/>
    <!-- parameters -->
    <xacro:arg name="tf_prefix" default="" />

File: src/eli_cs_robot_description/urdf/cs625.urdf.xacro (robot description, xacro)
@@ -1,4 +1,4 @@
 <?xml version="1.0"?>
-<robot xmlns:xacro="http://wiki.ros.org/xacro" name="$(arg name)">
+<robot xmlns:xacro="http://wiki.ros.org/xacro" name="cs625">
    <!-- robot name parameter -->
    <xacro:arg name="name" default="cs625"/>
@@ -7,5 +7,5 @@
    <!-- possible 'cs_type' values: cs63, cs66, cs612, cs616, cs620, cs625 -->
    <!-- the default value should raise an error in case this was called without defining the type -->
-   <xacro:arg name="cs_type" default="cs63"/>
+   <xacro:arg name="cs_type" default="cs625"/>
    <!-- parameters -->
    <xacro:arg name="tf_prefix" default="" />
@@ -113,4 +113,97 @@
      <origin xyz="-0.046 0 0.353" rpy="0 0 0"/>
    </joint>
+   <!-- ================================================================= -->
+   <!-- ==============  深度相机 (Depth Camera) ============== -->
+   <!-- ================================================================= -->
+   <link name="$(arg tf_prefix)camera_link">
+     <visual>
+       <origin xyz="0 0 0" rpy="0 0 0"/>
+       <geometry>
+         <box size="0.03 0.05 0.02"/>
+       </geometry>
+       <material name="camera_color">
+         <color rgba="0.2 0.2 0.2 1.0"/>
+       </material>
+     </visual>
+     <collision>
+       <origin xyz="0 0 0" rpy="0 0 0"/>
+       <geometry>
+         <box size="0.03 0.05 0.02"/>
+       </geometry>
+     </collision>
+     <inertial>
+       <mass value="0.05"/>
+       <inertia ixx="0.00001" ixy="0" ixz="0" iyy="0.00001" iyz="0" izz="0.00001"/>
+     </inertial>
+   </link>
+   <joint name="$(arg tf_prefix)camera_joint" type="fixed">
+     <parent link="$(arg tf_prefix)my_end_effector_link"/>
+     <child link="$(arg tf_prefix)camera_link"/>
+     <!-- Camera positioned 5cm in front of the EEF, pointing outward -->
+     <origin xyz="0.05 0 0.05" rpy="0 0.785 0"/>
+   </joint>
+   <!-- Ignition Gazebo RGBD camera sensor plugin -->
+   <xacro:if value="$(arg sim_ignition)">
+     <gazebo reference="$(arg tf_prefix)camera_link">
+       <sensor type="rgbd_camera" name="camera_sensor">
+         <pose>0 0 0 0 0 0</pose>
+         <always_on>1</always_on>
+         <update_rate>15.0</update_rate>
+         <topic>/camera</topic>
+         <camera>
+           <horizontal_fov>1.047</horizontal_fov>
+           <image>
+             <width>640</width>
+             <height>480</height>
+             <format>R8G8B8</format>
+           </image>
+           <clip>
+             <near>0.05</near>
+             <far>5.0</far>
+           </clip>
+         </camera>
+         <depth_camera>
+           <image>
+             <width>640</width>
+             <height>480</height>
+             <format>R_FLOAT32</format>
+           </image>
+           <clip>
+             <near>0.05</near>
+             <far>5.0</far>
+           </clip>
+         </depth_camera>
+       </sensor>
+     </gazebo>
+   </xacro:if>
+   <!-- Classic Gazebo RGBD camera sensor (fallback) -->
+   <xacro:if value="$(arg sim_gazebo)">
+     <gazebo reference="$(arg tf_prefix)camera_link">
+       <sensor type="depth_camera" name="camera_sensor">
+         <pose>0 0 0 0 0 0</pose>
+         <always_on>1</always_on>
+         <update_rate>15.0</update_rate>
+         <camera>
+           <horizontal_fov>1.047</horizontal_fov>
+           <image>
+             <width>640</width>
+             <height>480</height>
+             <format>R8G8B8</format>
+           </image>
+           <clip>
+             <near>0.05</near>
+             <far>5.0</far>
+           </clip>
+         </camera>
+         <plugin name="camera_depth_plugin" filename="libgazebo_ros_camera.so">
+           <ros>
+             <namespace>/camera</namespace>
+             <remapping>depth:=depth</remapping>
+             <remapping>points:=depth/points</remapping>
+           </ros>
+         </plugin>
+       </sensor>
+     </gazebo>
+   </xacro:if>
    <xacro:if value="$(arg sim_gazebo)">
     <!-- Gazebo plugins -->

File: src/eli_cs_robot_description/urdf/cs625_for_moveit.urdf (robot description, URDF)
Before this commit: robot cs625, 13 links, 12 joints
Joints:
- joint elbow_joint: origin xyz=-0.749559 0 0 rpy=0 0 0 -> xyz=-0.750517 0 0 rpy=0 0 0
- joint shoulder_lift_joint: origin xyz=0 0 0 rpy=1.570796326589793 0 0 -> xyz=0 0 0 rpy=1.5707999 0 0
- joint shoulder_pan_joint: origin xyz=0 0 0.227828 rpy=0 0 0 -> xyz=0 0 0.231007 rpy=0 0 0
- joint wrist_1_joint: origin xyz=-0.624488 0 0.173237 rpy=0 0 0 -> xyz=-0.623098 0 0.171144 rpy=0 0 0
- joint wrist_2_joint: origin xyz=0 -0.128407 0 rpy=1.570796326589793 0 0 -> xyz=0 -0.127906 0 rpy=1.5707999 0 0
- joint wrist_3_joint: origin xyz=0 0.128152 0 rpy=-1.570796326589793 0 0 -> xyz=0 0.127478 0 rpy=-1.5707999 0 0
